Commit message: feat: placo example

File: urdf/low_cost_robot.urdf (robot description, URDF)
Before this commit: robot low_cost_robot, 7 links, 6 joints
Links:
- link base_link: geometry collision mesh filename=file://urdf/meshes/base_link.stl scale=0.001 0.001 0.001; visual mesh filename=file://urdf/meshes/base_link.stl scale=0.001 0.001 0.001
- link gripper_moving_1: geometry collision mesh filename=file://urdf/meshes/gripper_moving_1.stl scale=0.001 0.001 0.001; visual mesh filename=file://urdf/meshes/gripper_moving_1.stl scale=0.001 0.001 0.001
- link gripper_static_1: geometry collision mesh filename=file://urdf/meshes/gripper_static_1.stl scale=0.001 0.001 0.001; visual mesh filename=file://urdf/meshes/gripper_static_1.stl scale=0.001 0.001 0.001
- link link1_1: geometry collision mesh filename=file://urdf/meshes/link1_1.stl scale=0.001 0.001 0.001; visual mesh filename=file://urdf/meshes/link1_1.stl scale=0.001 0.001 0.001
- link link2_1: geometry collision mesh filename=file://urdf/meshes/link2_1.stl scale=0.001 0.001 0.001; visual mesh filename=file://urdf/meshes/link2_1.stl scale=0.001 0.001 0.001
- link link3_1: geometry collision mesh filename=file://urdf/meshes/link3_1.stl scale=0.001 0.001 0.001; visual mesh filename=file://urdf/meshes/link3_1.stl scale=0.001 0.001 0.001
- link link4_1: geometry collision mesh filename=file://urdf/meshes/link4_1.stl scale=0.001 0.001 0.001; visual mesh filename=file://urdf/meshes/link4_1.stl scale=0.001 0.001 0.001

Commit message: feat: fix bug

File: urdf/low_cost_robot.urdf (robot description, URDF)
Before this commit: robot low_cost_robot, 7 links, 6 joints
Links:
- link base_link: geometry collision mesh filename=file://$(find low_cost_robot_description)/meshes/base_link.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 scale=0.001 0.001 0.001; visual mesh filename=file://$(find low_cost_robot_description)/meshes/base_link.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 scale=0.001 0.001 0.001
- link gripper_moving_1: geometry collision mesh filename=file://$(find low_cost_robot_description)/meshes/gripper_mo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 scale=0.001 0.001 0.001; visual mesh filename=file://$(find low_cost_robot_description)/meshes/gripper_mo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 scale=0.001 0.001 0.001
- link gripper_static_1: geometry collision mesh filename=file://$(find low_cost_robot_description)/meshes/gripper_st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 scale=0.001 0.001 0.001; visual mesh filename=file://$(find low_cost_robot_description)/meshes/gripper_st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 scale=0.001 0.001 0.001
- link link1_1: geometry collision mesh filename=file://$(find low_cost_robot_description)/meshes/link1_1.stl scale=0.001 0.001 0.001; visual mesh filename=file://$(find low_cost_robot_description)/meshes/link1_1.stl scale=0.001 0.001 0.001
- link link2_1: geometry collision mesh filename=file://$(find low_cost_robot_description)/meshes/link2_1.stl scale=0.001 0.001 0.001; visual mesh filename=file://$(find low_cost_robot_description)/meshes/link2_1.stl scale=0.001 0.001 0.001
- link link3_1: geometry collision mesh filename=file://$(find low_cost_robot_description)/meshes/link3_1.stl scale=0.001 0.001 0.001; visual mesh filename=file://$(find low_cost_robot_description)/meshes/link3_1.stl scale=0.001 0.001 0.001
- link link4_1: geometry collision mesh filename=file://$(find low_cost_robot_description)/meshes/link4_1.stl scale=0.001 0.001 0.001; visual mesh filename=file://$(find low_cost_robot_description)/meshes/link4_1.stl scale=0.001 0.001 0.001
